File: PCB/Aircopter.sch (EAGLE design)
At the start: 0 parts

Commit message: Update Schematic
Parts:
- added *1: STM32L432KCU6STM32L432KCU6_QFN32_5X5MM, Aircopter:STM32L432KCU6STM32L432KCU6_QFN32_5X5MM
- added *2: DSC6001CI1A-008.0000TDSC6001CI1A-008.0000T_VFLGA4, Aircopter:DSC6001CI1A-008.0000TDSC6001CI1A-008.0000T_VFLGA4
- added *3: TPS63001DRCRTPS63001DRCR_VSON10, Aircopter:TPS63001DRCRTPS63001DRCR_VSON10
Changed lines of the file:
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@@
 <grid distance="0.1" unitdist="inch" unit="inch" style="lines" multiple="1" display="no" altdistance="0.01" altunitdist="inch" altunit="inch"/>
 <layers>
+<layer number="1" name="Top" color="4" fill="1" visible="no" active="no"/>
+<layer number="2" name="Route2" color="1" fill="3" visible="no" active="no"/>
+<layer number="3" name="Route3" color="4" fill="3" visible="no" active="no"/>
+<layer number="4" name="Route4" color="1" fill="4" visible="no" active="no"/>
+<layer number="5" name="Route5" color="4" fill="4" visible="no" active="no"/>
+<layer number="6" name="Route6" color="1" fill="8" visible="no" active="no"/>
+<layer number="7" name="Route7" color="4" fill="8" visible="no" active="no"/>
+<layer number="8" name="Route8" color="1" fill="2" visible="no" active="no"/>
+<layer number="9" name="Route9" color="4" fill="2" visible="no" active="no"/>
+<layer number="10" name="Route10" color="1" fill="7" visible="no" active="no"/>
+<layer number="11" name="Route11" color="4" fill="7" visible="no" active="no"/>
+<layer number="12" name="Route12" color="1" fill="5" visible="no" active="no"/>
+<layer number="13" name="Route13" color="4" fill="5" visible="no" active="no"/>
+<layer number="14" name="Route14" color="1" fill="6" visible="no" active="no"/>
+<layer number="15" name="Route15" color="4" fill="6" visible="no" active="no"/>
+<layer number="16" name="Bottom" color="1" fill="1" visible="no" active="no"/>
+<layer number="17" name="Pads" color="2" fill="1" visible="no" active="no"/>
+<layer number="18" name="Vias" color="2" fill="1" visible="no" active="no"/>
+<layer number="19" name="Unrouted" color="6" fill="1" visible="no" active="no"/>
+<layer number="20" name="Dimension" color="15" fill="1" visible="no" active="no"/>
+<layer number="21" name="tPlace" color="7" fill="1" visible="no" active="no"/>
+<layer number="22" name="bPlace" color="7" fill="1" visible="no" active="no"/>
+<layer number="23" name="tOrigins" color="15" fill="1" visible="no" active="no"/>
+<layer number="24" name="bOrigins" color="15" fill="1" visible="no" active="no"/>
+<layer number="25" name="tNames" color="7" fill="1" visible="no" active="no"/>
+<layer number="26" name="bNames" color="7" fill="1" visible="no" active="no"/>
+<layer number="27" name="tValues" color="7" fill="1" visible="no" active="no"/>
+<layer number="28" name="bValues" color="7" fill="1" visible="no" active="no"/>
+<layer number="29" name="tStop" color="7" fill="3" visible="no" active="no"/>
+<layer number="30" name="bStop" color="7" fill="6" visible="no" active="no"/>
+<layer number="31" name="tCream" color="7" fill="4" visible="no" active="no"/>
+<layer number="32" name="bCream" color="7" fill="5" visible="no" active="no"/>
+<layer number="33" name="tFinish" color="6" fill="3" visible="no" active="no"/>
+<layer number="34" name="bFinish" color="6" fill="6" visible="no" active="no"/>
+<layer number="35" name="tGlue" color="7" fill="4" visible="no" active="no"/>
+<layer number="36" name="bGlue" color="7" fill="5" visible="no" active="no"/>
+<layer number="37" name="tTest" color="7" fill="1" visible="no" active="no"/>
+<layer number="38" name="bTest" color="7" fill="1" visible="no" active="no"/>
+<layer number="39" name="tKeepout" color="4" fill="11" visible="no" active="no"/>
+<layer number="40" name="bKeepout" color="1" fill="11" visible="no" active="no"/>
+<layer number="41" name="tRestrict" color="4" fill="10" visible="no" active="no"/>
+<layer number="42" name="bRestrict" color="1" fill="10" visible="no" active="no"/>
+<layer number="43" name="vRestrict" color="2" fill="10" visible="no" active="no"/>
+<layer number="44" name="Drills" color="7" fill="1" visible="no" active="no"/>
+<layer number="45" name="Holes" color="7" fill="1" visible="no" active="no"/>
+<layer number="46" name="Milling" color="3" fill="1" visible="no" active="no"/>
+<layer number="47" name="Measures" color="7" fill="1" visible="no" active="no"/>
+<layer number="48" name="Document" color="7" fill="1" visible="no" active="no"/>
+<layer number="49" name="Reference" color="7" fill="1" visible="no" active="no"/>
+<layer number="51" name="tDocu" color="7" fill="1" visible="no" active="no"/>
+<layer number="52" name="bDocu" color="7" fill="1" visible="no" active="no"/>
 <layer number="88" name="SimResults" color="9" fill="1" visible="yes" active="yes"/>
 <layer number="89" name="SimProbes" color="9" fill="1" visible="yes" active="yes"/>
@@
 </classes>
 <parts>
+<part name="*1" library="Aircopter" library_urn="urn:adsk.eagle:library:7112503" deviceset="STM32L432KCU6" device="STM32L432KCU6_QFN32_5X5MM" package3d_urn="urn:adsk.eagle:package:7112519/1"/>
+<part name="*2" library="Aircopter" library_urn="urn:adsk.eagle:library:7112503" deviceset="DSC6001CI1A-008.0000T" device="DSC6001CI1A-008.0000T_VFLGA4" package3d_urn="urn:adsk.eagle:package:7112517/1"/>
+<part name="*3" library="Aircopter" library_urn="urn:adsk.eagle:library:7112503" deviceset="TPS63001DRCR" device="TPS63001DRCR_VSON10" package3d_urn="urn:adsk.eagle:package:7112518/1"/>
 </parts>
 <sheets>
@@
 </plain>
 <instances>
+<instance part="*1" gate="A" x="20.32" y="55.88" smashed="yes">
+<attribute name="NAME" x="21.59" y="57.15" size="1.27" layer="95"/>
+<attribute name="VALUE" x="19.05" y="3.81" size="1.27" layer="96"/>
+</instance>
+<instance part="*2" gate="A" x="104.14" y="48.26" smashed="yes">
+<attribute name="NAME" x="102.87" y="49.53" size="1.27" layer="95"/>
+<attribute name="VALUE" x="87.63" y="41.91" size="1.27" layer="96"/>
+</instance>
+<instance part="*3" gate="A" x="99.06" y="27.94" smashed="yes">
+<attribute name="NAME" x="97.79" y="29.21" size="1.27" layer="95"/>
+<attribute name="VALUE" x="90.17" y="11.43" size="1.27" layer="96"/>
+</instance>
 </instances>
 <busses>
@@
 </schematic>
 </drawing>
+<compatibility>
+<note version="8.2" severity="warning">
+Since Version 8.2, EAGLE supports online libraries. The ids
+of those online libraries will not be understood (or retained)
+with this version.
+</note>
+<note version="8.3" severity="warning">
+Since Version 8.3, EAGLE supports URNs for individual library
+assets (packages, symbols, and devices). The URNs of those assets
+will not be understood (or retained) with this version.
+</note>
+<note version="8.3" severity="warning">
+Since Version 8.3, EAGLE supports the association of 3D packages
+with devices in libraries, schematics, and board files. Those 3D
+packages will not be understood (or retained) with this version.
+</note>
+</compatibility>
 </eagle>

Commit message: Update Sch
Parts:
- added C1, C2, C3, C4, C5, C6, C7, C8: (no value), rcl:C-USC0603K
- added J1: FTDI_DEVICE, AP_quad:FTDI_DEVICE
- added M1: WIRELESS-NRF24L01, AP_quad:WIRELESS-NRF24L01
- added P1: (no value), jst-ph:JST-PH2
- added U$1, U$2, U$3, U$4: N-CHANNEL-MOSFET-IRLML6244TRPBF, AP_quad:N-CHANNEL-MOSFET-IRLML6244TRPBF
- added U1: GY-521MPU6050, AP_quad:GY-521MPU6050
- *1: value STM32L432KCU6STM32L432KCU6_QFN32_5X5MM -> STM32L432KCU6
- *2: value DSC6001CI1A-008.0000TDSC6001CI1A-008.0000T_VFLGA4 -> DSC6001CI1A-008.0000T
- *3: value TPS63001DRCRTPS63001DRCR_VSON10 -> TPS63001DRCR

Commit message: Laid out voltage regular subcircuit
Parts:
- added *4: TPS63001DRCRTPS63001DRCR_VSON10, Aircopter:TPS63001DRCRTPS63001DRCR_VSON10
- added C11, C12, C13, C9: (no value), rcl:C-US025-025X050
- added L1: (no value), rcl:L-US0204/5
- added R1: (no value), rcl:R-US_R0603
- *3: value TPS63001DRCR -> TPS63001DRCRTPS63001DRCR_VSON10
Connections:
- new net GND: *4.EPAD/PGND, *4.GND, *4.PGND, C11.2, C12.2, C13.2, C9.2
- new net N$2: *4.L1, L1.2
- new net N$4: *4.L2, L1.1
- new net N$5: *4.EN, *4.PS/SYNC, *4.VINA, C11.1, R1.2
- new net VIN: *4.VIN, C9.1, R1.1
- new net VOUT: *4.FB, *4.VOUT, C12.1, C13.1
Other:
- note added: "GND and PGND must both be connected on the PCB at only one point, ideally close to the GND pin"

Commit message: Voltage regulator and battery subcircuit
Parts:
- removed C13: (no value), rcl:C-US025-025X050
- removed P1: (no value), jst-ph:JST-PH2
- added P2: (no value), jst-ph:JST-PH2
- C11: value (none) -> 100n
- C12: value (none) -> 33u
- C9: value (none) -> 10u
- L1: value (none) -> 1.5u
- R1: value (none) -> 100
Connections:
- removed net VOUT: *4.FB, *4.VOUT, C12.1, C13.1
- new net +3V3: *4.FB, *4.VOUT, C12.1
- net GND: now also P2.2; no longer C13.2
- net VIN: now also P2.1
Changed lines of the file:
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@@
 <part name="*2" library="Aircopter" library_urn="urn:adsk.eagle:library:7112503" deviceset="DSC6001CI1A-008.0000T" device="DSC6001CI1A-008.0000T_VFLGA4" package3d_urn="urn:adsk.eagle:package:7112517/1" value="DSC6001CI1A-008.0000T"/>
 <part name="FRAME1" library="frames" library_urn="urn:adsk.eagle:library:229" deviceset="DINA4_L" device=""/>
-<part name="SUPPLY1" library="supply2" library_urn="urn:adsk.eagle:library:372" deviceset="GND" device=""/>
-<part name="P1" library="jst-ph" deviceset="JST-PH2" device=""/>
 <part name="C1" library="rcl" library_urn="urn:adsk.eagle:library:334" deviceset="C-US" device="C0603K" package3d_urn="urn:adsk.eagle:package:23680/2"/>
 <part name="C2" library="rcl" library_urn="urn:adsk.eagle:library:334" deviceset="C-US" device="C0603K" package3d_urn="urn:adsk.eagle:package:23680/2"/>
@@
 <part name="*4" library="Aircopter" deviceset="TPS63001DRCR" device="TPS63001DRCR_VSON10"/>
 <part name="FRAME2" library="frames" library_urn="urn:adsk.eagle:library:229" deviceset="A3L-LOC" device=""/>
-<part name="L1" library="rcl" library_urn="urn:adsk.eagle:library:334" deviceset="L-US" device="0204/5" package3d_urn="urn:adsk.eagle:package:23488/1"/>
-<part name="R1" library="rcl" library_urn="urn:adsk.eagle:library:334" deviceset="R-US_" device="R0603" package3d_urn="urn:adsk.eagle:package:23555/2"/>
-<part name="C11" library="rcl" library_urn="urn:adsk.eagle:library:334" deviceset="C-US" device="025-025X050" package3d_urn="urn:adsk.eagle:package:23629/2"/>
-<part name="C12" library="rcl" library_urn="urn:adsk.eagle:library:334" deviceset="C-US" device="025-025X050" package3d_urn="urn:adsk.eagle:package:23629/2"/>
-<part name="C13" library="rcl" library_urn="urn:adsk.eagle:library:334" deviceset="C-US" device="025-025X050" package3d_urn="urn:adsk.eagle:package:23629/2"/>
-<part name="C9" library="rcl" library_urn="urn:adsk.eagle:library:334" deviceset="C-US" device="025-025X050" package3d_urn="urn:adsk.eagle:package:23629/2"/>
+<part name="L1" library="rcl" library_urn="urn:adsk.eagle:library:334" deviceset="L-US" device="0204/5" package3d_urn="urn:adsk.eagle:package:23488/1" value="1.5u"/>
+<part name="R1" library="rcl" library_urn="urn:adsk.eagle:library:334" deviceset="R-US_" device="R0603" package3d_urn="urn:adsk.eagle:package:23555/2" value="100"/>
+<part name="C11" library="rcl" library_urn="urn:adsk.eagle:library:334" deviceset="C-US" device="025-025X050" package3d_urn="urn:adsk.eagle:package:23629/2" value="100n"/>
+<part name="C12" library="rcl" library_urn="urn:adsk.eagle:library:334" deviceset="C-US" device="025-025X050" package3d_urn="urn:adsk.eagle:package:23629/2" value="33u"/>
+<part name="C9" library="rcl" library_urn="urn:adsk.eagle:library:334" deviceset="C-US" device="025-025X050" package3d_urn="urn:adsk.eagle:package:23629/2" value="10u"/>
+<part name="P2" library="jst-ph" deviceset="JST-PH2" device=""/>
+<part name="SUPPLY2" library="supply2" library_urn="urn:adsk.eagle:library:372" deviceset="GND" device=""/>
+<part name="+3V1" library="supply1" library_urn="urn:adsk.eagle:library:371" deviceset="+3V3" device=""/>
+<part name="SUPPLY1" library="supply2" library_urn="urn:adsk.eagle:library:372" deviceset="GND" device=""/>
+<part name="FRAME3" library="frames" library_urn="urn:adsk.eagle:library:229" deviceset="DINA4_L" device=""/>
 </parts>
 <sheets>
@@
 <attribute name="SHEET" x="248.92" y="1.27" size="2.54" layer="94"/>
 <attribute name="DRAWING_NAME" x="180.34" y="19.05" size="2.54" layer="94"/>
-</instance>
-<instance part="SUPPLY1" gate="GND" x="22.86" y="160.02" smashed="yes">
-<attribute name="VALUE" x="20.955" y="156.845" size="1.778" layer="96"/>
-</instance>
-<instance part="P1" gate="G$1" x="12.7" y="167.64" smashed="yes">
-<attribute name="NAME" x="10.16" y="170.942" size="1.778" layer="95"/>
-<attribute name="VALUE" x="10.16" y="160.274" size="1.778" layer="96"/>
 </instance>
 <instance part="C1" gate="G$1" x="7.62" y="78.74" smashed="yes">
@@
 <attribute name="VALUE" x="125.476" y="117.729" size="1.778" layer="96"/>
 </instance>
-<instance part="C13" gate="G$1" x="132.08" y="121.92" smashed="yes">
-<attribute name="NAME" x="136.144" y="123.825" size="1.778" layer="95" rot="R180"/>
-<attribute name="VALUE" x="133.096" y="117.729" size="1.778" layer="96"/>
-</instance>
 <instance part="C9" gate="G$1" x="33.02" y="104.14" smashed="yes">
 <attribute name="NAME" x="34.036" y="104.775" size="1.778" layer="95"/>
 <attribute name="VALUE" x="34.036" y="99.949" size="1.778" layer="96"/>
+</instance>
+<instance part="P2" gate="G$1" x="12.7" y="124.46" smashed="yes">
+<attribute name="NAME" x="10.16" y="127.762" size="1.778" layer="95"/>
+<attribute name="VALUE" x="10.16" y="117.094" size="1.778" layer="96"/>
+</instance>
+<instance part="SUPPLY2" gate="GND" x="22.86" y="116.84" smashed="yes">
+<attribute name="VALUE" x="20.955" y="113.665" size="1.778" layer="96"/>
+</instance>
+<instance part="+3V1" gate="G$1" x="144.78" y="132.08" smashed="yes">
+<attribute name="VALUE" x="142.24" y="127" size="1.778" layer="96" rot="R90"/>
+</instance>
+<instance part="SUPPLY1" gate="GND" x="45.72" y="91.44" smashed="yes">
+<attribute name="VALUE" x="43.815" y="88.265" size="1.778" layer="96"/>
 </instance>
 </instances>
@@
 </busses>
 <nets>
-<net name="VOUT" class="0">
-<segment>
-<pinref part="*4" gate="A" pin="VOUT"/>
-<wire x1="114.3" y1="124.46" x2="116.84" y2="124.46" width="0.1524" layer="91"/>
-<pinref part="*4" gate="A" pin="FB"/>
-<wire x1="116.84" y1="124.46" x2="124.46" y2="124.46" width="0.1524" layer="91"/>
-<wire x1="124.46" y1="124.46" x2="132.08" y2="124.46" width="0.1524" layer="91"/>
-<wire x1="132.08" y1="124.46" x2="142.24" y2="124.46" width="0.1524" layer="91"/>
-<wire x1="114.3" y1="119.38" x2="116.84" y2="119.38" width="0.1524" layer="91"/>
-<wire x1="116.84" y1="119.38" x2="116.84" y2="124.46" width="0.1524" layer="91"/>
-<junction x="116.84" y="124.46"/>
-<pinref part="C13" gate="G$1" pin="1"/>
-<junction x="132.08" y="124.46"/>
-<pinref part="C12" gate="G$1" pin="1"/>
-<junction x="124.46" y="124.46"/>
-<label x="142.24" y="124.46" size="1.778" layer="95" xref="yes"/>
-</segment>
-</net>
 <net name="VIN" class="0">
 <segment>
@@
 <wire x1="45.72" y1="119.38" x2="45.72" y2="124.46" width="0.1524" layer="91"/>
 <junction x="45.72" y="124.46"/>
-<label x="20.32" y="124.46" size="1.778" layer="95" rot="R180" xref="yes"/>
+<pinref part="P2" gate="G$1" pin="1"/>
 </segment>
 </net>
@@
 <wire x1="33.02" y1="96.52" x2="45.72" y2="96.52" width="0.1524" layer="91"/>
 <junction x="45.72" y="96.52"/>
-<label x="45.72" y="93.98" size="1.778" layer="95" rot="R270" xref="yes"/>
 <pinref part="*4" gate="A" pin="PGND"/>
 <wire x1="114.3" y1="109.22" x2="116.84" y2="109.22" width="0.1524" layer="91"/>
@@
 <wire x1="124.46" y1="114.3" x2="124.46" y2="116.84" width="0.1524" layer="91"/>
 <junction x="116.84" y="114.3"/>
-<wire x1="124.46" y1="114.3" x2="132.08" y2="114.3" width="0.1524" layer="91"/>
-<wire x1="132.08" y1="114.3" x2="132.08" y2="116.84" width="0.1524" layer="91"/>
-<junction x="124.46" y="114.3"/>
-<pinref part="C13" gate="G$1" pin="2"/>
 <pinref part="C12" gate="G$1" pin="2"/>
 <wire x1="45.72" y1="96.52" x2="116.84" y2="96.52" width="0.1524" layer="91"/>
 <wire x1="116.84" y1="96.52" x2="116.84" y2="106.68" width="0.1524" layer="91"/>
 <junction x="116.84" y="106.68"/>
+<pinref part="SUPPLY1" gate="GND" pin="GND"/>
+</segment>
+<segment>
+<pinref part="P2" gate="G$1" pin="2"/>
+<wire x1="20.32" y1="121.92" x2="22.86" y2="121.92" width="0.1524" layer="91"/>
+<pinref part="SUPPLY2" gate="GND" pin="GND"/>
+<wire x1="22.86" y1="121.92" x2="22.86" y2="119.38" width="0.1524" layer="91"/>
+</segment>
+</net>
+<net name="+3V3" class="0">
+<segment>
+<pinref part="*4" gate="A" pin="VOUT"/>
+<wire x1="114.3" y1="124.46" x2="116.84" y2="124.46" width="0.1524" layer="91"/>
+<pinref part="*4" gate="A" pin="FB"/>
+<wire x1="116.84" y1="124.46" x2="124.46" y2="124.46" width="0.1524" layer="91"/>
+<wire x1="124.46" y1="124.46" x2="144.78" y2="124.46" width="0.1524" layer="91"/>
+<wire x1="114.3" y1="119.38" x2="116.84" y2="119.38" width="0.1524" layer="91"/>
+<wire x1="116.84" y1="119.38" x2="116.84" y2="124.46" width="0.1524" layer="91"/>
+<junction x="116.84" y="124.46"/>
+<pinref part="C12" gate="G$1" pin="1"/>
+<junction x="124.46" y="124.46"/>
+<pinref part="+3V1" gate="G$1" pin="+3V3"/>
+<wire x1="144.78" y1="124.46" x2="144.78" y2="129.54" width="0.1524" layer="91"/>
 </segment>
 </net>
 </nets>
 </sheet>
+<sheet>
+<plain>
+</plain>
+<instances>
+<instance part="FRAME3" gate="G$1" x="0" y="0" smashed="yes"/>
+<instance part="FRAME3" gate="G$2" x="162.56" y="0" smashed="yes">
+<attribute name="LAST_DATE_TIME" x="175.26" y="1.27" size="2.54" layer="94"/>
+<attribute name="SHEET" x="248.92" y="1.27" size="2.54" layer="94"/>
+<attribute name="DRAWING_NAME" x="180.34" y="19.05" size="2.54" layer="94"/>
+</instance>
+</instances>
+<busses>
+</busses>
+<nets>
+</nets>
+</sheet>

Commit message: Finish Schematic
Parts:
- removed *3: TPS63001DRCRTPS63001DRCR_VSON10, Aircopter:TPS63001DRCRTPS63001DRCR_VSON10
- added C10, C15: 100n, rcl:C-USC0603K
- added C13: 10u, rcl:C-USC0603K
- added C14: 100u, rcl:C-US025-025X050
- added P1, P3, P4, P5: (no value), jst-ph:JST-PH2
- added R2, R3, R4, R5: 10k, resistor:R-US_R0603
- added R6: (no value), resistor:R-US_R0603
- added S1: SWITCH-MOMENTARY-2SMD, AP_quad:SWITCH-MOMENTARY-2SMD
- added SV1: (no value), con-lstb:MA04-1
- added U$5, U$7: IRLML6244TRPBF, AP_quad:N-CHANNEL-MOSFET-IRLML6244TRPBF
- added U$6, U$8: DB2W40300L, AP_quad:DB2W40300L
- C1, C3, C4, C7: value (none) -> 100n
- C2: value (none) -> 10p\
- C5: value (none) -> 4.7u
- C6: value (none) -> 10n
- C8: value (none) -> 1u
- U$1, U$3: value N-CHANNEL-MOSFET-IRLML6244TRPBF -> DB2W40300L; device AP_quad:N-CHANNEL-MOSFET-IRLML6244TRPBF -> AP_quad:DB2W40300L
- U$2, U$4: value N-CHANNEL-MOSFET-IRLML6244TRPBF -> IRLML6244TRPBF
Connections:
- new net CTS: *1.PA11, J1.CTS
- new net MISO: *1.PA6, M1.MISO
- new net MOSI: *1.PA7, M1.MOSI
- new net MOTOR1: *1.PA8, R2.2, U$5.G
- new net MOTOR2: *1.PA1, R3.2, U$2.G
- new net MOTOR3: *1.PA2, R4.2, U$4.G
- new net MOTOR4: *1.PA3, R5.2, U$7.G
- new net N$1: P3.1, U$1.PPIN, U$5.D
- new net N$12: C3.2, C4.2, C5.2
- new net N$3: P1.1, U$2.D, U$3.PPIN
- new net N$6: P4.1, U$4.D, U$6.PPIN
- new net N$7: P5.1, U$7.D, U$8.PPIN
- new net NRST: *1.NRST, C15.1, R6.1, S1.1, SV1.1
- new net NSS: *1.PA4, M1.CSN
- new net OSC: *1.PA0/CK_IN, *2.OUT, C2.1
- new net RADIO_CE: *1.PB0, M1.CE
- new net RTS: *1.PA12, J1.DTR
- new net RX: *1.PA10, J1.TXO
- new net SCK: *1.PA5, M1.SCK
- new net SCL: *1.PB6, U1.SCL
- new net SDA: *1.PB7, U1.SDA
- new net SWCLK: *1.PA14, SV1.4
- new net SWDIO: *1.PA13, SV1.2
- new net TX: *1.PA9, J1.RXI
- net +3V3: now also *1.VDD@1, *1.VDD@2, *1.VDDA/VREF+, *2.OE/STBY/FS, *2.VDD, C1.1, C10.1, C13.1, C3.1, C4.1, C5.1, C6.1, C7.1, C8.1, J1.VCC, M1.VCC, P1.2, P3.2, P4.2, P5.2, R6.2, U$1.GPIN, U$3.GPIN, U$6.GPIN, U$8.GPIN, U1.VCC
- net GND: now also *1.VSS@1, *1.VSS@2, *1.VSS@3, *2.GND, C1.2, C10.2, C13.2, C14.2, C15.2, C2.2, C6.2, C7.2, C8.2, J1.GND, M1.GND, R2.1, R3.1, R4.1, R5.1, S1.2, SV1.3, U$2.S, U$4.S, U$5.S, U$7.S, U1.ADO, U1.GND
- net VIN: now also C14.1
Other:
- note added: "MCU"
- note added: "MCU VDD Decoupling Capacitors"
- note added: "MCU VDDA Decoupling Capacitors"
- note added: "Oscillator"
- note added: "Programmer"
- note added: "Radio"
- note added: "Reset"
- note added: "UART/FTDI"

Commit message: Finish Schematic
Parts:
- added R7, R8: 100k, rcl:R-US_R0603
Connections:
- new net BATSENSE: *1.PB1, R7.2, R8.1
- net GND: now also R8.2
- net VIN: now also R7.1
Other:
- moved on the sheet: *4, C1, C11, C12, C14, C15, C2, C9, L1, P2, R1, R6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
