File: PCB/Aircopter.brd (EAGLE design)
At the start: 28 x 47 mm, 46 parts, among them J1 FTDI_DEVICE, M1 WIRELESS-NRF24L01, U1 GY-521MPU6050

Commit message: Mid-design review PCB updates
Parts:
- moved C13 0.48 mm to (4.88, 2.90)
- moved C10 0.48 mm to (6.38, 2.95)
- moved R7 0.20 mm to (14.3, 21.0)
- moved C3 0.13 mm to (16.3, 25.9)
- moved C4 0.07 mm to (10.1, 33.5), turned to 45 degrees
